File: KiCad/CPU.kicad_pcb (KiCad board)
At the start: 2 copper layers, 102.8 x 73.8 mm, 9 parts, among them J1 Conn_02x08_Odd_Even, J2 Conn_02x08_Odd_Even, J3 Conn_02x08_Odd_Even, J4 Conn_02x09_Odd_Even, J5 Bus_ISA_8bit, J6 Raspberry_Pi_2_3, J7 Conn_02x02_Counter_Clockwise

Commit message: started new pcb design
Parts:
- removed J7: Conn_02x02_Counter_Clockwise, Connector_PinHeader_2.54mm:PinHeader_2x02_P2.54mm_Vertical
- added C1: 0.1u, Capacitor_SMD:C_0603_1608Metric, F.Cu at (184.0, 67.5)
- added J66: Conn_02x08_Odd_Even, Connector_PinHeader_2.54mm:PinHeader_2x08_P2.54mm_Vertical, F.Cu at (183.0, 98.0)
- added R2: 10k, Resistor_SMD:R_0603_1608Metric, F.Cu at (187.0, 92.9)
- added R3: 10k, Resistor_SMD:R_0603_1608Metric, F.Cu at (187.0, 87.8)
- added R4: 10k, Resistor_SMD:R_0603_1608Metric, F.Cu at (187.0, 82.8)
- added R5: 10k, Resistor_SMD:R_0603_1608Metric, F.Cu at (187.0, 80.2)
- added R6: 10k, Resistor_SMD:R_0603_1608Metric, F.Cu at (187.0, 85.3)
- added R7: 10k, Resistor_SMD:R_0603_1608Metric, F.Cu at (187.0, 90.4)
- added R8: 10k, Resistor_SMD:R_0603_1608Metric, F.Cu at (187.0, 95.5)
- added U19: 74LS688, Package_DIP:DIP-20_W7.62mm_Socket, F.Cu at (165.0, 100.0)
- R1: value 100 -> 10k
- moved R1 30.8 mm to (187.0, 98.0), turned to 180 degrees
Connections:
- CS1 pad 1: unconnected-(CS1-Pad1) -> GND
- CS1 pad 2: Net-(CS1-Pad2) -> V3
- CS1 pad 3: VCC -> SPDIF_OUT
- J1 pad 10: ~{DACK1} -> IRQ4
- J1 pad 12: CLK -> A10
- J1 pad 2: PCM_OUT -> OSC
- J1 pad 4: PCM_FS -> CLK
- J1 pad 6: PCM_CLK -> A11
- J1 pad 8: DRQ1 -> IRQ3
- J2 pad 15: RP22 -> ROM
- J3 pad 1: IRQ3 -> IRQ5
- J3 pad 3: IRQ4 -> IRQ7
- J3 pad 5: IRQ5 -> IRQ1
- J3 pad 7: IRQ6 -> DRQ1
- J3 pad 9: IRQ7 -> ~{DACK1}
- J5 pad 19: unconnected-(J5-Pad19) -> IRQ1
- J5 pad 22: IRQ6 -> unconnected-(J5-Pad22)
- J5 pad 30: unconnected-(J5-Pad30) -> OSC
- J5 pad 43: unconnected-(J5-Pad43) -> A19
- J5 pad 44: unconnected-(J5-Pad44) -> A18
- J5 pad 45: unconnected-(J5-Pad45) -> A17
- J5 pad 46: unconnected-(J5-Pad46) -> A16
- J5 pad 47: unconnected-(J5-Pad47) -> A15
- J5 pad 48: unconnected-(J5-Pad48) -> A14
- J5 pad 49: unconnected-(J5-Pad49) -> A13
- J5 pad 50: unconnected-(J5-Pad50) -> A12
- J5 pad 51: unconnected-(J5-Pad51) -> A11
- J5 pad 52: unconnected-(J5-Pad52) -> A10
- J6 pad 12: PCM_CLK -> unconnected-(J6-Pad12)
- J6 pad 22: RP22 -> unconnected-(J6-Pad22)
- J6 pad 35: PCM_FS -> unconnected-(J6-Pad35)
- J6 pad 40: PCM_OUT -> unconnected-(J6-Pad40)
- R1 pad 1: SPDIF_OUT -> VCC
- R1 pad 2: Net-(CS1-Pad2) -> R0
Routing:
- net A12: track 0.00 -> 105.4 mm, vias 0 -> 2
- net A13: track 0.00 -> 94.3 mm, vias 0 -> 2
- net A14: track 0.00 -> 83.1 mm, vias 0 -> 2
- net A15: track 0.00 -> 72.7 mm, vias 0 -> 2
- net PCM_CLK: track 71.6 -> 0.00 mm
- net PCM_FS: track 62.9 -> 0.00 mm
- net ROM: track 0.00 -> 60.4 mm, vias 0 -> 2
- net A16: track 0.00 -> 59.1 mm, vias 0 -> 2
- net PCM_OUT: track 54.1 -> 0.00 mm
- net A17: track 0.00 -> 53.9 mm, vias 0 -> 2
- net A18: track 0.00 -> 49.8 mm, vias 0 -> 2
- net A19: track 0.00 -> 41.8 mm, vias 0 -> 2
- net V3: track 45.8 -> 82.4 mm
- net AEN: track 19.1 -> 53.9 mm, vias 0 -> 2
- net A11: track 0.00 -> 33.7 mm
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