File: KiCad/CPU.kicad_sch (KiCad schematic)
At the start: 9 parts, among them J1 Conn_02x08_Odd_Even, J2 Conn_02x08_Odd_Even, J3 Conn_02x08_Odd_Even, J4 Conn_02x09_Odd_Even, J5 Bus_ISA_8bit, J6 Raspberry_Pi_2_3, J7 Conn_02x02_Counter_Clockwise

Commit message: started new pcb design
Parts:
- removed J7: Conn_02x02_Counter_Clockwise, Connector_PinHeader_2.54mm:PinHeader_2x02_P2.54mm_Vertical, symbol Connector_Generic:Conn_02x02_Counter_Clockwise
- added C1: (no value), symbol pspice:C
- added J66: Conn_02x08_Odd_Even, Connector_PinHeader_2.54mm:PinHeader_2x08_P2.54mm_Vertical, symbol Connector_Generic:Conn_02x08_Odd_Even
- added R2, R3, R4, R5, R6, R7, R8: 10k, Resistor_SMD:R_0603_1608Metric, symbol Device:R
- added U19: (no value), symbol 74xx:74LS688
- CS1: value (none) -> TOTX1350_F_; footprint (none) -> TOTX1350F
- J2, J3: value Conn_02x08_Odd_Even -> (none); footprint Connector_PinHeader_2.54mm:PinHeader_2x08_P2.54mm_Vertical -> (none)
- R1: value (none) -> 10k; footprint (none) -> Resistor_SMD:R_0603_1608Metric
- renumbered J5 to J7
Connections:
- net AEN: now also U19.1 (G)
- net CLK: now also J1.4 (Pin_4); no longer J1.12 (Pin_12)
- net DRQ1: now also J3.7 (Pin_7); no longer J1.8 (Pin_8)
- net GND: now also CS1.1 (NC_1), C1.2, J66.1 (Pin_1), J66.11 (Pin_11), J66.13 (Pin_13), J66.15 (Pin_15), J66.3 (Pin_3), J66.5 (Pin_5), J66.7 (Pin_7), J66.9 (Pin_9), U19.10 (GND)
- net IRQ3: now also J1.8 (Pin_8); no longer J3.1 (Pin_1)
- net IRQ4: now also J1.10 (Pin_10); no longer J3.3 (Pin_3)
- net IRQ5: now also J3.1 (Pin_1); no longer J3.5 (Pin_5)
- net IRQ7: now also J3.3 (Pin_3); no longer J3.9 (Pin_9)
- net SPDIF_OUT: now also CS1.3 (ANODE); no longer R1.1
- net V3: now also CS1.2 (CATHODE), C1.1
- net VCC: now also R1.1, R2.1, R3.1, R4.1, R5.1, R6.1, R7.1, R8.1, U19.20 (VCC); no longer CS1.3 (ANODE)
- net ~{DACK1}: now also J3.9 (Pin_9); no longer J1.10 (Pin_10)
- net IRQ1: now reaches J7.19 (~{DACK0})
- net IRQ1: now also J3.5 (Pin_5)
- net OSC: now reaches J7.30 (OSC)
- net OSC: now also J1.2 (Pin_2)
- net A19: now reaches J7.43 (BA19)
- net A19: now also U19.17 (P7)
- net A18: now reaches J7.44 (BA18)
- net A18: now also U19.15 (P6)
- net A17: now reaches J7.45 (BA17)
- net A17: now also U19.13 (P5)
- net A16: now reaches J7.46 (BA16)
- net A16: now also U19.11 (P4)
- net A15: now reaches J7.47 (BA15)
- net A15: now also U19.8 (P3)
- net A14: now reaches J7.48 (BA14)
- net A14: now also U19.6 (P2)
- net A13: now reaches J7.49 (BA13)
- net A13: now also U19.4 (P1)
- net A12: now reaches J7.50 (BA12)
- net A12: now also U19.2 (P0)
- net A11: now reaches J7.51 (BA11)
- net A11: now also J1.6 (Pin_6)
- net A10: now reaches J7.52 (BA10)
- net A10: now also J1.12 (Pin_12)
- net R0: now reaches R1.2
- net R0: now also J66.2 (Pin_2), U19.3 (R0); no longer CS1.2 (CATHODE)
- net IRQ6: no longer names the net of J7.22 (IRQ6)
- net IRQ6: no longer J3.7 (Pin_7)
- net PCM_CLK: no longer names the net of J6.12 (GPIO18/PWM0)
- net PCM_CLK: no longer J1.6 (Pin_6)
- net PCM_FS: no longer names the net of J6.35 (GPIO19/MISO1)
- net PCM_FS: no longer J1.4 (Pin_4)
- net PCM_OUT: no longer names the net of J6.40 (GPIO21/SCLK1)
- net PCM_OUT: no longer J1.2 (Pin_2)
- net RP22: no longer names the net of J6.22 (GPIO25)
- net RP22: no longer J2.15 (Pin_15)
- new net R1: J66.6 (Pin_6), R2.2, U19.5 (R1)
- new net R2: J66.10 (Pin_10), R3.2, U19.7 (R2)
- new net R3: J66.14 (Pin_14), R4.2, U19.9 (R3)
- new net R4: J66.16 (Pin_16), R5.2, U19.12 (R4)
- new net R5: J66.12 (Pin_12), R6.2, U19.14 (R5)
- new net R6: J66.8 (Pin_8), R7.2, U19.16 (R6)
- new net R7: J66.4 (Pin_4), R8.2, U19.18 (R7)
- new net ROM: J2.15 (Pin_15), U19.19 (P=R)
- no-connect marks 25 -> 13
Other:
- note added: "* DMA1 is the only DMA channel available (due to lack of pins) * IRQ6 is NC, but IRQ1 is connected to REFRESH (custom MOBO uses to control PIC-board)"
- note added: "PLAN -Use 12 address bits directly -Use 74LS688 for ROM -Connect OSC PIN -Fix TOSLINK"
- note removed: "* IRQ7, DACK1 and DRQ1 are used when acting as Sound Blaster (IRQ & DMA) * IRQ6 can be used by keyboard with our CPU-board"
